Commit message: errors resolved, code modules combined into one stable version.

File: robot.urdf (robot description, URDF)
Before this commit: robot moveo_urdf, 13 links, 12 joints
Joints:
- joint Gripper_Idol_Gear_Joint: limit lower=-1.5707 upper=0 effort=5 velocity=1 -> lower=-0.75 upper=0 effort=5 velocity=1; mimic (none) -> joint=Gripper_Servo_Gear_Joint multiplier=-1 offset=0
- joint Gripper_Servo_Gear_Joint: limit lower=0 upper=1.5707 effort=5 velocity=1 -> lower=0 upper=0.75 effort=5 velocity=1
- joint Tip_Gripper_Idol_Joint: limit lower=-1.5 upper=0 effort=5 velocity=1 -> lower=-0.75 upper=0 effort=5 velocity=1; mimic joint=Gripper_Idol_Gear_Joint multiplier=-1 offset=0 -> joint=Gripper_Idol_Gear_Joint multiplier=1 offset=0
- joint Tip_Gripper_Servo_Joint: limit lower=0 upper=1.3 effort=5 velocity=1 -> lower=0 upper=0.75 effort=5 velocity=1; type continuous -> revolute

Commit message: upgrade of the scene env. gripper issues resolved

File: robot.urdf (robot description, URDF)
Before this commit: robot moveo_urdf, 13 links, 12 joints
Joints:
- joint Gripper_Idol_Gear_Joint: limit lower=-0.75 upper=0 effort=5 velocity=1 -> lower=-0.85 upper=0 effort=5 velocity=1
- joint Gripper_Servo_Gear_Joint: limit lower=0 upper=0.75 effort=5 velocity=1 -> lower=0 upper=0.85 effort=5 velocity=1
- joint Tip_Gripper_Idol_Joint: limit lower=-0.75 upper=0 effort=5 velocity=1 -> lower=0 upper=0.85 effort=5 velocity=1; mimic joint=Gripper_Idol_Gear_Joint multiplier=1 offset=0 -> joint=Pivot_Arm_Gripper_Idol_Joint multiplier=-1 offset=0; origin xyz=-0.039906 -0.000125 -0.0027473 rpy=3.1416 0.5236 3.1416 -> xyz=0.047000399 -0.0002497656 -0.020000514 rpy=-1.4354494E-05 -0.45484816 1.5077933E-05; parent Gripper_Idol_Gear -> Pivot_Arm_Gripper_Idol
- joint Tip_Gripper_Servo_Joint: limit lower=0 upper=0.75 effort=5 velocity=1 -> lower=0 upper=0.85 effort=5 velocity=1; mimic joint=Gripper_Servo_Gear_Joint multiplier=1 offset=0 -> joint=Pivot_Arm_Gripper_Servo_Joint multiplier=1 offset=0; origin xyz=-0.039906 -0.004 -0.0027473 rpy=-3.1416 -1.5569 -2.0392E-12 -> xyz=-0.047278677 0.00029943856 -0.019899708 rpy=-3.1415187 -1.4881423 -6.4581482E-05; parent Gripper_Servo_Gear -> Pivot_Arm_Gripper_Servo
